Commit message: Add ethercat hardware interface.

File: hiwin_ra6_moveit_config/config/ecat.ros2_control.xacro (robot description, xacro)
@@ -1,33 +1,27 @@
 <?xml version="1.0"?>
 <robot xmlns:xacro="http://www.ros.org/wiki/xacro">
-  <xacro:macro name="ecat_ros2_control"
-    params="name tf_prefix control_frequency">
-    <xacro:property name="pb4d_config"
-      value="$(find hiwin_driver)/config/SANYO_PB4D_config.yaml" />
+  <xacro:macro name="ecat_ros2_control" params="name ra_type tf_prefix">
+    <xacro:property name="joint_1_config" value="$(find hiwin_driver)/config/${ra_type}/joint_1_config.yaml" />
+    <xacro:property name="joint_2_config" value="$(find hiwin_driver)/config/${ra_type}/joint_2_config.yaml" />
+    <xacro:property name="joint_3_config" value="$(find hiwin_driver)/config/${ra_type}/joint_3_config.yaml" />
+    <xacro:property name="joint_4_config" value="$(find hiwin_driver)/config/${ra_type}/joint_4_config.yaml" />
+    <xacro:property name="joint_5_config" value="$(find hiwin_driver)/config/${ra_type}/joint_5_config.yaml" />
+    <xacro:property name="joint_6_config" value="$(find hiwin_driver)/config/${ra_type}/joint_6_config.yaml" />
     <ros2_control name="ecat" type="system">
       <hardware>
         <plugin>ethercat_driver/EthercatDriver</plugin>
         <param name="master_id">0</param>
-        <param name="control_frequency">${control_frequency}</param>
+        <param name="control_frequency">1000</param>
       </hardware>
-      <joint name="mdp_device">
-        <ec_module name="device_1">
-          <plugin>ethercat_generic_plugins/EcMDPDevice</plugin>
-          <param name="alias">0</param>
-          <param name="position">0</param>
-          <param name="slave_config">${pb4d_config}</param>
-        </ec_module>
-      </joint>
       <joint name="${tf_prefix}joint_1">
         <command_interface name="position" />
         <state_interface name="position" />
         <state_interface name="velocity" />
-        <ec_module name="module_1">
-          <plugin>ethercat_generic_plugins/EcMDPModule</plugin>
+        <ec_module name="RS3">
+          <plugin>ethercat_generic_plugins/EcCiA402Drive</plugin>
           <param name="alias">0</param>
           <param name="position">0</param>
-          <param name="axis">1</param>
           <param name="mode_of_operation">8</param>
-          <param name="slave_config">${pb4d_config}</param>
+          <param name="slave_config">${joint_1_config}</param>
         </ec_module>
       </joint>
@@ -36,11 +30,10 @@
         <state_interface name="position" />
         <state_interface name="velocity" />
-        <ec_module name="module_2">
-          <plugin>ethercat_generic_plugins/EcMDPModule</plugin>
+        <ec_module name="RS3">
+          <plugin>ethercat_generic_plugins/EcCiA402Drive</plugin>
           <param name="alias">0</param>
-          <param name="position">0</param>
-          <param name="axis">2</param>
+          <param name="position">1</param>
           <param name="mode_of_operation">8</param>
-          <param name="slave_config">${pb4d_config}</param>
+          <param name="slave_config">${joint_2_config}</param>
         </ec_module>
       </joint>
@@ -49,11 +42,10 @@
         <state_interface name="position" />
         <state_interface name="velocity" />
-        <ec_module name="module_3">
-          <plugin>ethercat_generic_plugins/EcMDPModule</plugin>
+        <ec_module name="RS3">
+          <plugin>ethercat_generic_plugins/EcCiA402Drive</plugin>
           <param name="alias">0</param>
-          <param name="position">0</param>
-          <param name="axis">3</param>
+          <param name="position">2</param>
           <param name="mode_of_operation">8</param>
-          <param name="slave_config">${pb4d_config}</param>
+          <param name="slave_config">${joint_3_config}</param>
         </ec_module>
       </joint>
@@ -62,35 +54,35 @@
         <state_interface name="position" />
         <state_interface name="velocity" />
-        <ec_module name="module_4">
-          <plugin>ethercat_generic_plugins/EcMDPModule</plugin>
+        <ec_module name="RS3">
+          <plugin>ethercat_generic_plugins/EcCiA402Drive</plugin>
           <param name="alias">0</param>
-          <param name="position">0</param>
-          <param name="axis">4</param>
+          <param name="position">3</param>
           <param name="mode_of_operation">8</param>
-          <param name="slave_config">${pb4d_config}</param>
+          <param name="slave_config">${joint_4_config}</param>
         </ec_module>
       </joint>
-    </ros2_control>
-    <ros2_control name="fake" type="system">
-      <hardware>
-        <plugin>mock_components/GenericSystem</plugin>
-      </hardware>
       <joint name="${tf_prefix}joint_5">
         <command_interface name="position" />
-        <state_interface name="position">
-          <param name="initial_value">0.0</param>
-        </state_interface>
-        <state_interface name="velocity">
-          <param name="initial_value">0.0</param>
-        </state_interface>
+        <state_interface name="position" />
+        <state_interface name="velocity" />
+        <ec_module name="RS3">
+          <plugin>ethercat_generic_plugins/EcCiA402Drive</plugin>
+          <param name="alias">0</param>
+          <param name="position">4</param>
+          <param name="mode_of_operation">8</param>
+          <param name="slave_config">${joint_5_config}</param>
+        </ec_module>
       </joint>
       <joint name="${tf_prefix}joint_6">
         <command_interface name="position" />
-        <state_interface name="position">
-          <param name="initial_value">0.0</param>
-        </state_interface>
-        <state_interface name="velocity">
-          <param name="initial_value">0.0</param>
-        </state_interface>
+        <state_interface name="position" />
+        <state_interface name="velocity" />
+        <ec_module name="RS3">
+          <plugin>ethercat_generic_plugins/EcCiA402Drive</plugin>
+          <param name="alias">0</param>
+          <param name="position">5</param>
+          <param name="mode_of_operation">8</param>
+          <param name="slave_config">${joint_6_config}</param>
+        </ec_module>
       </joint>
     </ros2_control>

File: hiwin_ra6_moveit_config/config/ra6.urdf.xacro (robot description, xacro)
@@ -11,5 +11,4 @@
     <xacro:arg name="cabinet" default="gc2" />
     <xacro:arg name="robot_ip" default="0.0.0.0" />
-    <xacro:arg name="control_frequency" default="1000" />
     <xacro:property name="controller" value="$(arg cabinet)" />
     <xacro:property name="hardware_name" value="FakeSystem" />
@@ -32,6 +31,6 @@
     </xacro:if>
     <xacro:if value="${controller == 'ecat'}">
-        <xacro:ecat_ros2_control name="${hardware_name}" tf_prefix="$(arg tf_prefix)"
-            control_frequency="$(arg control_frequency)" />
+        <xacro:ecat_ros2_control name="${hardware_name}" ra_type="$(arg ra_type)"
+            tf_prefix="$(arg tf_prefix)" />
     </xacro:if>
 </robot>

Commit message: implement IO hardware interface using GPIO and isolated IO

File: hiwin_ra6_moveit_config/config/ecat.ros2_control.xacro (robot description, xacro)
@@ -12,5 +12,5 @@
         <plugin>ethercat_driver/EthercatDriver</plugin>
         <param name="master_id">0</param>
-        <param name="control_frequency">1000</param>
+        <param name="control_frequency">500</param>
       </hardware>
       <joint name="${tf_prefix}joint_1">
@@ -87,4 +87,63 @@
       </joint>
     </ros2_control>
+    <ros2_control name="GPIO" type="system">
+      <hardware>
+        <plugin>hiwin_driver/HIWINGPIOHardwareInterface</plugin>
+      </hardware>
+      <gpio name="system">
+        <command_interface name="watchdog" />
+        <command_interface name="reset_safety_rly" />
+        <command_interface name="reset_driver" />
+        <state_interface name="breaker" />
+        <state_interface name="e_stop" />
+        <state_interface name="e_stop2" />
+        <state_interface name="fan_error" />
+        <state_interface name="capacitor_error" />
+        <state_interface name="clear_error_notify" />
+        <state_interface name="shutdown_notify" />
+      </gpio>
+      <gpio name="digital">
+        <command_interface name="DO1" />
+        <command_interface name="DO2" />
+        <command_interface name="DO3" />
+        <command_interface name="DO4" />
+        <command_interface name="DO5" />
+        <command_interface name="DO6" />
+        <command_interface name="DO7" />
+        <command_interface name="DO8" />
+        <state_interface name="DI1" />
+        <state_interface name="DI2" />
+        <state_interface name="DI3" />
+        <state_interface name="DI4" />
+        <state_interface name="DI5" />
+        <state_interface name="DI6" />
+        <state_interface name="DI7" />
+        <state_interface name="DI8" />
+      </gpio>
+      <gpio name="robot">
+        <command_interface name="VO1" />
+        <command_interface name="VO2" />
+        <command_interface name="VO3" />
+        <command_interface name="VO_EN1" />
+        <command_interface name="VO_EN2" />
+        <command_interface name="VO_EN3" />
+        <command_interface name="RO1" />
+        <command_interface name="RO2" />
+        <command_interface name="RO3" />
+        <command_interface name="RO4" />
+        <command_interface name="RO5" />
+        <command_interface name="RO6" />
+        <command_interface name="RO7" />
+        <command_interface name="RO8" />
+        <state_interface name="RI1" />
+        <state_interface name="RI2" />
+        <state_interface name="RI3" />
+        <state_interface name="RI4" />
+        <state_interface name="RI5" />
+        <state_interface name="RI6" />
+        <state_interface name="RI7" />
+        <state_interface name="RI8" />
+      </gpio>
+    </ros2_control>
   </xacro:macro>
 </robot>

File: hiwin_rs4_moveit_config/config/ecat.ros2_control.xacro (robot description, xacro)
@@ -1,19 +1,14 @@
 <?xml version="1.0"?>
 <robot xmlns:xacro="http://www.ros.org/wiki/xacro">
-  <xacro:macro name="ecat_ros2_control"
-    params="name rs_type tf_prefix">
-    <xacro:property name="joint_1_config"
-      value="$(find hiwin_driver)/config/${rs_type}/joint_1_config.yaml" />
-    <xacro:property name="joint_2_config"
-      value="$(find hiwin_driver)/config/${rs_type}/joint_2_config.yaml" />
-    <xacro:property name="joint_3_config"
-      value="$(find hiwin_driver)/config/${rs_type}/joint_3_config.yaml" />
-    <xacro:property name="joint_4_config"
-      value="$(find hiwin_driver)/config/${rs_type}/joint_4_config.yaml" />
-    <ros2_control name="ecat" type="system">
+  <xacro:macro name="ecat_ros2_control" params="name rs_type tf_prefix">
+    <xacro:property name="joint_1_config" value="$(find hiwin_driver)/config/${rs_type}/joint_1_config.yaml" />
+    <xacro:property name="joint_2_config" value="$(find hiwin_driver)/config/${rs_type}/joint_2_config.yaml" />
+    <xacro:property name="joint_3_config" value="$(find hiwin_driver)/config/${rs_type}/joint_3_config.yaml" />
+    <xacro:property name="joint_4_config" value="$(find hiwin_driver)/config/${rs_type}/joint_4_config.yaml" />
+    <ros2_control name="${name}" type="system">
       <hardware>
         <plugin>ethercat_driver/EthercatDriver</plugin>
         <param name="master_id">0</param>
-        <param name="control_frequency">1000</param>
+        <param name="control_frequency">500</param>
       </hardware>
       <joint name="${tf_prefix}joint_1">
@@ -66,4 +61,39 @@
       </joint>
     </ros2_control>
+    <ros2_control name="GPIO" type="system">
+      <hardware>
+        <plugin>hiwin_driver/HIWINGPIOHardwareInterface</plugin>
+      </hardware>
+      <gpio name="system">
+        <command_interface name="watchdog" />
+        <command_interface name="reset_safety_rly" />
+        <command_interface name="reset_driver" />
+        <state_interface name="breaker" />
+        <state_interface name="e_stop" />
+        <state_interface name="e_stop2" />
+        <state_interface name="fan_error" />
+        <state_interface name="capacitor_error" />
+        <state_interface name="clear_error_notify" />
+        <state_interface name="shutdown_notify" />
+      </gpio>
+      <gpio name="digital">
+        <command_interface name="DO1" />
+        <command_interface name="DO2" />
+        <command_interface name="DO3" />
+        <command_interface name="DO4" />
+        <command_interface name="DO5" />
+        <command_interface name="DO6" />
+        <command_interface name="DO7" />
+        <command_interface name="DO8" />
+        <state_interface name="DI1" />
+        <state_interface name="DI2" />
+        <state_interface name="DI3" />
+        <state_interface name="DI4" />
+        <state_interface name="DI5" />
+        <state_interface name="DI6" />
+        <state_interface name="DI7" />
+        <state_interface name="DI8" />
+      </gpio>
+    </ros2_control>
   </xacro:macro>
 </robot>
