Commit message: Implement control robot

File: hiwin_ra6_moveit_config/config/ra6.ros2_control.xacro (robot description, xacro)
@@ -1,11 +1,17 @@
 <?xml version="1.0"?>
 <robot xmlns:xacro="http://www.ros.org/wiki/xacro">
-  <xacro:macro name="ra6_ros2_control" params="name tf_prefix initial_positions_file">
+  <xacro:macro name="ra6_ros2_control"
+    params="name tf_prefix initial_positions_file use_fake_hardware robot_ip">
     <xacro:property name="initial_positions"
       value="${xacro.load_yaml(initial_positions_file)['initial_positions']}" />
     <ros2_control name="${name}" type="system">
       <hardware>
-        <!-- By default, set up controllers for simulation. This won't work on real hardware -->
-        <plugin>mock_components/GenericSystem</plugin>
+        <xacro:if value="${use_fake_hardware}">
+          <plugin>mock_components/GenericSystem</plugin>
+        </xacro:if>
+        <xacro:unless value="${use_fake_hardware}">
+          <plugin>hiwin_driver/HIWINPositionHardwareInterface</plugin>
+          <param name="robot_ip">${robot_ip}</param>
+        </xacro:unless>
       </hardware>
       <joint name="${tf_prefix}joint_1">

File: hiwin_ra6_moveit_config/config/ra6.urdf.xacro (robot description, xacro)
@@ -1,11 +1,25 @@
 <?xml version="1.0"?>
 <robot xmlns:xacro="http://www.ros.org/wiki/xacro" name="ra6">
+    <xacro:arg name="tf_prefix" default="" />
     <xacro:arg name="initial_positions_file"
         default="$(find hiwin_ra6_moveit_config)/config/initial_positions.yaml" />
     <!-- Import ra6 urdf file -->
+    <xacro:arg name="ra_type" default="ra6x" />
     <xacro:include filename="$(find hiwin_description)/urdf/ra.urdf.xacro" />
     <!-- Import control_xacro -->
-    <xacro:include filename="$(find hiwin_ra6_moveit_config)/config/ra6.ros2_control.xacro" />
-    <xacro:ra6_ros2_control name="FakeSystem" tf_prefix="$(arg tf_prefix)"
-        initial_positions_file="$(arg initial_positions_file)" />
+    <xacro:arg name="use_fake_hardware" default="false" />
+    <xacro:arg name="hardware_file" default="ra6.ros2_control.xacro" />
+    <xacro:arg name="robot_ip" default="0.0.0.0" />
+    <xacro:property name="hardware" value="$(arg hardware_file)" />
+    <xacro:property name="hardware_name" value="FakeSystem" />
+    <xacro:unless value="$(arg use_fake_hardware)">
+        <xacro:if value="${hardware == 'ra6.ros2_control.xacro'}">
+            <xacro:property name="hardware_name" value="GC2" />
+        </xacro:if>
+    </xacro:unless>
+    <xacro:include filename="$(find hiwin_ra6_moveit_config)/config/$(arg hardware_file)" />
+    <xacro:ra6_ros2_control name="${hardware_name}" tf_prefix="$(arg tf_prefix)"
+        initial_positions_file="$(arg initial_positions_file)"
+        use_fake_hardware="$(arg use_fake_hardware)"
+        robot_ip="$(arg robot_ip)" />
 </robot>

Commit message: update YAML config and launch files for IO hardware interface

File: hiwin_ra6_moveit_config/config/ra6.ros2_control.xacro (robot description, xacro)
@@ -1,8 +1,6 @@
 <?xml version="1.0"?>
 <robot xmlns:xacro="http://www.ros.org/wiki/xacro">
-  <xacro:macro name="ra6_ros2_control"
-    params="name tf_prefix initial_positions_file use_fake_hardware robot_ip">
-    <xacro:property name="initial_positions"
-      value="${xacro.load_yaml(initial_positions_file)['initial_positions']}" />
+  <xacro:macro name="ra6_ros2_control" params="name tf_prefix initial_positions_file use_fake_hardware robot_ip">
+    <xacro:property name="initial_positions" value="${xacro.load_yaml(initial_positions_file)['initial_positions']}" />
     <ros2_control name="${name}" type="system">
       <hardware>

File: hiwin_ra6_moveit_config/config/ra6.urdf.xacro (robot description, xacro)
@@ -2,6 +2,5 @@
 <robot xmlns:xacro="http://www.ros.org/wiki/xacro" name="ra6">
     <xacro:arg name="tf_prefix" default="" />
-    <xacro:arg name="initial_positions_file"
-        default="$(find hiwin_ra6_moveit_config)/config/initial_positions.yaml" />
+    <xacro:arg name="initial_positions_file" default="$(find hiwin_ra6_moveit_config)/config/initial_positions.yaml" />
     <!-- Import ra6 urdf file -->
     <xacro:arg name="ra_type" default="ra6x" />
@@ -25,12 +24,8 @@
     <xacro:include filename="$(find hiwin_ra6_moveit_config)/config/${hardware_description_file}" />
     <xacro:if value="${controller == 'gc2'}">
-        <xacro:ra6_ros2_control name="${hardware_name}" tf_prefix="$(arg tf_prefix)"
-            initial_positions_file="$(arg initial_positions_file)"
-            use_fake_hardware="$(arg use_fake_hardware)"
-            robot_ip="$(arg robot_ip)" />
+        <xacro:ra6_ros2_control name="${hardware_name}" tf_prefix="$(arg tf_prefix)" initial_positions_file="$(arg initial_positions_file)" use_fake_hardware="$(arg use_fake_hardware)" robot_ip="$(arg robot_ip)" />
     </xacro:if>
     <xacro:if value="${controller == 'ecat'}">
-        <xacro:ecat_ros2_control name="${hardware_name}" ra_type="$(arg ra_type)"
-            tf_prefix="$(arg tf_prefix)" />
+        <xacro:ecat_ros2_control name="${hardware_name}" ra_type="$(arg ra_type)" tf_prefix="$(arg tf_prefix)" />
     </xacro:if>
 </robot>

File: hiwin_rs4_moveit_config/config/rs4.ros2_control.xacro (robot description, xacro)
@@ -1,8 +1,6 @@
 <?xml version="1.0"?>
 <robot xmlns:xacro="http://www.ros.org/wiki/xacro">
-  <xacro:macro name="rs4_ros2_control"
-    params="name tf_prefix initial_positions_file use_fake_hardware robot_ip">
-    <xacro:property name="initial_positions"
-      value="${xacro.load_yaml(initial_positions_file)['initial_positions']}" />
+  <xacro:macro name="rs4_ros2_control" params="name tf_prefix initial_positions_file use_fake_hardware robot_ip">
+    <xacro:property name="initial_positions" value="${xacro.load_yaml(initial_positions_file)['initial_positions']}" />
     <ros2_control name="${name}" type="system">
       <hardware>

File: hiwin_rs4_moveit_config/config/rs4.urdf.xacro (robot description, xacro)
@@ -2,6 +2,5 @@
 <robot xmlns:xacro="http://www.ros.org/wiki/xacro" name="rs4">
     <xacro:arg name="tf_prefix" default="" />
-    <xacro:arg name="initial_positions_file"
-        default="$(find hiwin_rs4_moveit_config)/config/initial_positions.yaml" />
+    <xacro:arg name="initial_positions_file" default="$(find hiwin_rs4_moveit_config)/config/initial_positions.yaml" />
     <!-- Import rs4 urdf file -->
     <xacro:arg name="rs_type" default="rs4x" />
@@ -9,5 +8,5 @@
     <!-- Import control_xacro -->
     <xacro:arg name="use_fake_hardware" default="false" />
-    <xacro:arg name="cabinet" default="gc2" />
+    <xacro:arg name="cabinet" default="rc4-a" />
     <xacro:arg name="robot_ip" default="0.0.0.0" />
     <xacro:property name="controller" value="$(arg cabinet)" />
@@ -25,12 +24,8 @@
     <xacro:include filename="$(find hiwin_rs4_moveit_config)/config/${hardware_description_file}" />
     <xacro:if value="${controller == 'rc4-a'}">
-        <xacro:rs4_ros2_control name="${hardware_name}" tf_prefix="$(arg tf_prefix)"
-            initial_positions_file="$(arg initial_positions_file)"
-            use_fake_hardware="$(arg use_fake_hardware)"
-            robot_ip="$(arg robot_ip)" />
+        <xacro:rs4_ros2_control name="${hardware_name}" tf_prefix="$(arg tf_prefix)" initial_positions_file="$(arg initial_positions_file)" use_fake_hardware="$(arg use_fake_hardware)" robot_ip="$(arg robot_ip)" />
     </xacro:if>
     <xacro:if value="${controller == 'ecat'}">
-        <xacro:ecat_ros2_control name="${hardware_name}" rs_type="$(arg rs_type)"
-            tf_prefix="$(arg tf_prefix)" />
+        <xacro:ecat_ros2_control name="${hardware_name}" rs_type="$(arg rs_type)" tf_prefix="$(arg tf_prefix)" />
     </xacro:if>
 </robot>
