Commit message: Add ethercat hardware interface.

File: hiwin_rs4_moveit_config/config/pb4.ros2_control.xacro (robot description, xacro)
@@ -2,29 +2,32 @@
 <robot xmlns:xacro="http://www.ros.org/wiki/xacro">
   <xacro:macro name="ecat_ros2_control"
-    params="name rs_type tf_prefix">
-    <xacro:property name="joint_1_config"
-      value="$(find hiwin_driver)/config/${rs_type}/joint_1_config.yaml" />
-    <xacro:property name="joint_2_config"
-      value="$(find hiwin_driver)/config/${rs_type}/joint_2_config.yaml" />
-    <xacro:property name="joint_3_config"
-      value="$(find hiwin_driver)/config/${rs_type}/joint_3_config.yaml" />
-    <xacro:property name="joint_4_config"
-      value="$(find hiwin_driver)/config/${rs_type}/joint_4_config.yaml" />
+    params="name tf_prefix control_frequency">
+    <xacro:property name="pb4d_config"
+      value="$(find hiwin_driver)/config/SANYO_PB4D_config.yaml" />
     <ros2_control name="ecat" type="system">
       <hardware>
         <plugin>ethercat_driver/EthercatDriver</plugin>
         <param name="master_id">0</param>
-        <param name="control_frequency">1000</param>
+        <param name="control_frequency">${control_frequency}</param>
       </hardware>
+      <joint name="mdp_device">
+        <ec_module name="device_1">
+          <plugin>ethercat_generic_plugins/EcMDPDevice</plugin>
+          <param name="alias">0</param>
+          <param name="position">0</param>
+          <param name="slave_config">${pb4d_config}</param>
+        </ec_module>
+      </joint>
       <joint name="${tf_prefix}joint_1">
         <command_interface name="position" />
         <state_interface name="position" />
         <state_interface name="velocity" />
-        <ec_module name="D2COE">
-          <plugin>ethercat_generic_plugins/EcCiA402Drive</plugin>
+        <ec_module name="module_1">
+          <plugin>ethercat_generic_plugins/EcMDPModule</plugin>
           <param name="alias">0</param>
           <param name="position">0</param>
+          <param name="axis">1</param>
           <param name="mode_of_operation">8</param>
-          <param name="slave_config">${joint_1_config}</param>
+          <param name="slave_config">${pb4d_config}</param>
         </ec_module>
       </joint>
@@ -33,10 +36,11 @@
         <state_interface name="position" />
         <state_interface name="velocity" />
-        <ec_module name="D2COE">
-          <plugin>ethercat_generic_plugins/EcCiA402Drive</plugin>
+        <ec_module name="module_2">
+          <plugin>ethercat_generic_plugins/EcMDPModule</plugin>
           <param name="alias">0</param>
-          <param name="position">1</param>
+          <param name="position">0</param>
+          <param name="axis">2</param>
           <param name="mode_of_operation">8</param>
-          <param name="slave_config">${joint_2_config}</param>
+          <param name="slave_config">${pb4d_config}</param>
         </ec_module>
       </joint>
@@ -45,10 +49,11 @@
         <state_interface name="position" />
         <state_interface name="velocity" />
-        <ec_module name="D2COE">
-          <plugin>ethercat_generic_plugins/EcCiA402Drive</plugin>
+        <ec_module name="module_3">
+          <plugin>ethercat_generic_plugins/EcMDPModule</plugin>
           <param name="alias">0</param>
-          <param name="position">2</param>
+          <param name="position">0</param>
+          <param name="axis">3</param>
           <param name="mode_of_operation">8</param>
-          <param name="slave_config">${joint_3_config}</param>
+          <param name="slave_config">${pb4d_config}</param>
         </ec_module>
       </joint>
@@ -57,10 +62,11 @@
         <state_interface name="position" />
         <state_interface name="velocity" />
-        <ec_module name="D2COE">
-          <plugin>ethercat_generic_plugins/EcCiA402Drive</plugin>
+        <ec_module name="module_4">
+          <plugin>ethercat_generic_plugins/EcMDPModule</plugin>
           <param name="alias">0</param>
-          <param name="position">3</param>
+          <param name="position">0</param>
+          <param name="axis">4</param>
           <param name="mode_of_operation">8</param>
-          <param name="slave_config">${joint_4_config}</param>
+          <param name="slave_config">${pb4d_config}</param>
         </ec_module>
       </joint>

File: hiwin_rs4_moveit_config/config/rs4.urdf.xacro (robot description, xacro)
@@ -1,8 +1,8 @@
 <?xml version="1.0"?>
-<robot xmlns:xacro="http://www.ros.org/wiki/xacro" name="ra6">
+<robot xmlns:xacro="http://www.ros.org/wiki/xacro" name="rs4">
     <xacro:arg name="tf_prefix" default="" />
     <xacro:arg name="initial_positions_file"
         default="$(find hiwin_rs4_moveit_config)/config/initial_positions.yaml" />
-    <!-- Import ra6 urdf file -->
+    <!-- Import rs4 urdf file -->
     <xacro:arg name="rs_type" default="rs4x" />
     <xacro:include filename="$(find hiwin_description)/urdf/rs.urdf.xacro" />
@@ -11,11 +11,10 @@
     <xacro:arg name="cabinet" default="gc2" />
     <xacro:arg name="robot_ip" default="0.0.0.0" />
-    <xacro:arg name="control_frequency" default="1000" />
     <xacro:property name="controller" value="$(arg cabinet)" />
     <xacro:property name="hardware_name" value="FakeSystem" />
     <xacro:property name="hardware_description_file" value="rs4.ros2_control.xacro" />
     <xacro:unless value="$(arg use_fake_hardware)">
-        <xacro:if value="${controller == 'gc2'}">
-            <xacro:property name="hardware_name" value="GC2" />
+        <xacro:if value="${controller == 'rc4-a'}">
+            <xacro:property name="hardware_name" value="RC4-A" />
         </xacro:if>
         <xacro:if value="${controller == 'ecat'}">
@@ -25,5 +24,5 @@
     </xacro:unless>
     <xacro:include filename="$(find hiwin_rs4_moveit_config)/config/${hardware_description_file}" />
-    <xacro:if value="${controller == 'gc2'}">
+    <xacro:if value="${controller == 'rc4-a'}">
         <xacro:rs4_ros2_control name="${hardware_name}" tf_prefix="$(arg tf_prefix)"
             initial_positions_file="$(arg initial_positions_file)"
@@ -32,6 +31,6 @@
     </xacro:if>
     <xacro:if value="${controller == 'ecat'}">
-        <xacro:ecat_ros2_control name="${hardware_name}" tf_prefix="$(arg tf_prefix)"
-            control_frequency="$(arg control_frequency)" />
+        <xacro:ecat_ros2_control name="${hardware_name}" rs_type="$(arg rs_type)"
+            tf_prefix="$(arg tf_prefix)" />
     </xacro:if>
 </robot>
